File: kicad_files_ANSIFULL/m80_ansifull.kicad_pcb (KiCad board)
At the start: 2 copper layers, 347.1 x 136.9 mm, 0 parts

Commit message: ANSIFULL plate done
Parts:
- added GR1: Eighty plated logo, m80s_library:eighty_logo_17.6x8mm, F.Cu at (136.7, 151.2)
- added GR2: Gondo logo, gondolindrim_kicad_logos:gondolindrim_circuit-tree_10.4x12, F.Cu at (191.7, 151.7)
- added REF**: M2-COUNTERSUNK, m65_plates_library:M2_Countersunk, F.Cu at (369.3, 133.2)
- added REF**: M2-COUNTERSUNK, m65_plates_library:M2_Countersunk, F.Cu at (40.7, 63.2)
- added REF**: M2-COUNTERSUNK, m65_plates_library:M2_Countersunk, F.Cu at (150.3, 50.3)
- added REF**: MountingHole_2.2mm_M2_DIN965_Pad_TopBottom, MountingHole:MountingHole_2.2mm_M2_DIN965_Pad_TopBottom, F.Cu at (335.3, 164.4)
- added REF**: MountingHole_2.2mm_M2_DIN965_Pad_TopBottom, MountingHole:MountingHole_2.2mm_M2_DIN965_Pad_TopBottom, F.Cu at (75.1, 32.7)
- added REF**: MountingHole_2.2mm_M2_DIN965_Pad_TopBottom, MountingHole:MountingHole_2.2mm_M2_DIN965_Pad_TopBottom, F.Cu at (335.3, 32.7)
- added REF**: MountingHole_2.2mm_M2_DIN965_Pad_TopBottom, MountingHole:MountingHole_2.2mm_M2_DIN965_Pad_TopBottom, F.Cu at (248.6, 32.7)
- added REF**: M2-COUNTERSUNK, m65_plates_library:M2_Countersunk, F.Cu at (56.2, 152.3)
- added REF**: M2-COUNTERSUNK, m65_plates_library:M2_Countersunk, F.Cu at (236.0, 50.3)
- added REF**: MountingHole_2.2mm_M2_DIN965_Pad_TopBottom, MountingHole:MountingHole_2.2mm_M2_DIN965_Pad_TopBottom, F.Cu at (248.6, 164.4)
- added REF**: M2-COUNTERSUNK, m65_plates_library:M2_Countersunk, F.Cu at (202.8, 150.8)
- added REF**: MountingHole_2.2mm_M2_DIN965_Pad, MountingHole:MountingHole_2.2mm_M2_DIN965_Pad, F.Cu at (280.7, 63.2)
- added REF**: MountingHole_2.2mm_M2_DIN965_Pad_TopBottom, MountingHole:MountingHole_2.2mm_M2_DIN965_Pad_TopBottom, F.Cu at (75.1, 164.4)
- added REF**: MountingHole_2.2mm_M2_DIN965_Pad, MountingHole:MountingHole_2.2mm_M2_DIN965_Pad, F.Cu at (130.0, 63.2)
- added REF**: M2-COUNTERSUNK, m65_plates_library:M2_Countersunk, F.Cu at (328.3, 110.1)
- added REF**: MountingHole_2.2mm_M2_DIN965_Pad, MountingHole:MountingHole_2.2mm_M2_DIN965_Pad, F.Cu at (51.6, 63.2)
- added REF**: M2-COUNTERSUNK, m65_plates_library:M2_Countersunk, F.Cu at (369.3, 63.2)
- added REF**: MountingHole_2.2mm_M2_DIN965_Pad, MountingHole:MountingHole_2.2mm_M2_DIN965_Pad, F.Cu at (359.0, 63.2)
- added REF**: MountingHole_2.2mm_M2_DIN965_Pad_TopBottom, MountingHole:MountingHole_2.2mm_M2_DIN965_Pad_TopBottom, F.Cu at (161.8, 32.7)
Routing:
- added copper zone on B.Cu, net GND
- added copper zone on F.Cu, net GND
Other:
- board size 347.1 x 136.9 mm -> 347.1 x 137.5 mm
- board text added: "0.5"
- board text added: "1.1"
- board text added: "1.6"
- board text added: "2.2"
- board text added: "45 deg"
- board text added: "DFU: 5S"
- board text added: "M2 - COUNTERSUNK"
- board text added: "RESET: TAP"
- board text added: "UNITS: mm"
