File: kicad_files_ANSIFULL/m80_ansifull.kicad_pcb (KiCad board)
At the start: 2 copper layers, 347.1 x 137.5 mm, 21 parts

Commit message: New V3 outlines
Parts:
- removed the REF** at (280.7, 63.2)
- removed the REF** at (130.0, 63.2)
- added ?: , , F.Cu at (247.3, 63.2)
- added ?: , , F.Cu at (320.7, 63.2)
- added ?: , , F.Cu at (163.2, 63.2)
- added REF**: MountingHole_2.2mm_M2_DIN965_Pad, MountingHole:MountingHole_2.2mm_M2_DIN965_Pad, F.Cu at (89.8, 63.2)
