File: kicad_files_ANSIFULL/m80_ansifull.kicad_sch (KiCad schematic)
At the start: 0 parts

Commit message: ANSIFULL plate done
Parts:
- added R_DUMMY: 0, Resistor_SMD:R_0201_0603Metric, symbol Device:R_Small
Connections:
- new net GND: R_DUMMY.1, R_DUMMY.2
Other:
- note added: "Resistor added so that the PCB has a GND net."
Changed lines of the file:
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@@
 (kicad_sch (version 20210621) (generator eeschema)
   (paper "A4")
-  (symbol_instances)
+  (text "Resistor added so that the PCB has a GND net." (at 144.78 49.53 0)
+    (effects (font (size 1.27 1.27)) (justify left bottom))
+  )
+  (symbol (lib_id "power:GND") (at 151.13 53.34 180) (unit 1)
+    (in_bom yes) (on_board yes) (fields_autoplaced)
+    (property "Reference" "#PWR0101" (id 0) (at 151.13 46.99 0)
+      (effects (font (size 1.27 1.27)) hide)
+    )
+    (property "Value" "GND" (id 1) (at 153.67 52.2604 0)
+      (effects (font (size 1.27 1.27)) (justify right))
+    )
+    (property "Footprint" "" (id 2) (at 151.13 53.34 0)
+      (effects (font (size 1.27 1.27)) hide)
+    )
+    (property "Datasheet" "" (id 3) (at 151.13 53.34 0)
+      (effects (font (size 1.27 1.27)) hide)
+    )
+    (pin "1")
+  )
+  (symbol (lib_id "power:GND") (at 151.13 58.42 0) (unit 1)
+    (in_bom yes) (on_board yes) (fields_autoplaced)
+    (property "Reference" "#PWR01" (id 0) (at 151.13 64.77 0)
+      (effects (font (size 1.27 1.27)) hide)
+    )
+    (property "Value" "GND" (id 1) (at 151.13 63.5 0))
+    (property "Footprint" "" (id 2) (at 151.13 58.42 0)
+      (effects (font (size 1.27 1.27)) hide)
+    )
+    (property "Datasheet" "" (id 3) (at 151.13 58.42 0)
+      (effects (font (size 1.27 1.27)) hide)
+    )
+    (pin "1")
+  )
+  (symbol (lib_id "Device:R_Small") (at 151.13 55.88 0) (unit 1)
+    (in_bom yes) (on_board yes) (fields_autoplaced)
+    (property "Reference" "R_DUMMY" (id 0) (at 153.67 54.6099 0)
+      (effects (font (size 1.27 1.27)) (justify left))
+    )
+    (property "Value" "0" (id 1) (at 153.67 57.1499 0)
+      (effects (font (size 1.27 1.27)) (justify left))
+    )
+    (property "Footprint" "Resistor_SMD:R_0201_0603Metric" (id 2) (at 151.13 55.88 0)
+      (effects (font (size 1.27 1.27)) hide)
+    )
+    (property "Datasheet" "~" (id 3) (at 151.13 55.88 0)
+      (effects (font (size 1.27 1.27)) hide)
+    )
+    (pin "1")
+    (pin "2")
+  )
+  (sheet_instances
+    (path "/" (page "1"))
+  )
+  (symbol_instances
+    (path "/9fbd5009-e7ae-403c-8bde-6ee102e13a86"
+      (reference "#PWR01") (unit 1) (value "GND") (footprint "")
+    )
+    (path "/3023c3c8-59de-4c42-b577-74cb0277597a"
+      (reference "#PWR0101") (unit 1) (value "GND") (footprint "")
+    )
+    (path "/456b4e56-d06b-4ba6-9fa1-2eb35a6173d0"
+      (reference "R_DUMMY") (unit 1) (value "0") (footprint "Resistor_SMD:R_0201_0603Metric")
+    )
+  )
 )
