File: kicad_files_ANSIHALF/m80_ansihalf.kicad_pcb (KiCad board)
At the start: 2 copper layers, 347.1 x 137.5 mm, 13 parts

Commit message: New V3 outlines
Parts:
- removed the REF** at (127.3, 62.3)
- removed the REF** at (278.0, 62.3)
- added ?: , , F.Cu at (160.4, 62.3)
- added ?: , , F.Cu at (244.6, 62.3)
- added ?: , , F.Cu at (318.0, 62.3)
- added REF**: MountingHole_2.2mm_M2_DIN965_Pad, MountingHole:MountingHole_2.2mm_M2_DIN965_Pad, F.Cu at (87.1, 62.3)
