File: kicad_files_UNIVERSALFULL/m80_universalfull.kicad_pcb (KiCad board)
At the start: 2 copper layers, 347.1 x 137.5 mm, 21 parts

Commit message: New V3 outlines
Parts:
- removed the REF** at (37.1, 59.2)
- removed the REF** at (71.5, 160.5)
- removed the REF** at (331.8, 160.5)
- removed the REF** at (245.0, 160.5)
- removed the REF** at (232.5, 46.4)
- removed the REF** at (52.7, 148.3)
- removed the REF** at (355.5, 59.2)
- removed the REF** at (365.8, 129.3)
- removed the REF** at (277.1, 59.2)
- removed the REF** at (158.3, 28.7)
- removed the REF** at (324.8, 106.2)
- removed the REF** at (331.8, 28.7)
- removed the REF** at (71.5, 28.7)
- removed the REF** at (146.7, 46.3)
- removed the REF** at (48.1, 59.2)
- removed the REF** at (245.0, 28.7)
- removed the REF** at (199.3, 146.8)
- removed the REF** at (365.8, 59.2)
- removed the REF** at (126.4, 59.2)
- added ?: , , F.Cu at (247.3, 63.2)
- added ?: , , F.Cu at (163.2, 63.2)
- added ?: , , F.Cu at (320.7, 63.2)
- added REF**: M2-COUNTERSUNK, m65_plates_library:M2_Countersunk, F.Cu at (369.3, 133.2)
- added REF**: M2-COUNTERSUNK, m65_plates_library:M2_Countersunk, F.Cu at (150.3, 50.3)
- added REF**: MountingHole_2.2mm_M2_DIN965_Pad_TopBottom, MountingHole:MountingHole_2.2mm_M2_DIN965_Pad_TopBottom, F.Cu at (335.3, 164.4)
- added REF**: MountingHole_2.2mm_M2_DIN965_Pad_TopBottom, MountingHole:MountingHole_2.2mm_M2_DIN965_Pad_TopBottom, F.Cu at (75.1, 32.7)
- added REF**: MountingHole_2.2mm_M2_DIN965_Pad_TopBottom, MountingHole:MountingHole_2.2mm_M2_DIN965_Pad_TopBottom, F.Cu at (335.3, 32.7)
- added REF**: MountingHole_2.2mm_M2_DIN965_Pad_TopBottom, MountingHole:MountingHole_2.2mm_M2_DIN965_Pad_TopBottom, F.Cu at (248.6, 32.7)
- added REF**: M2-COUNTERSUNK, m65_plates_library:M2_Countersunk, F.Cu at (56.2, 152.3)
- added REF**: M2-COUNTERSUNK, m65_plates_library:M2_Countersunk, F.Cu at (236.0, 50.3)
- added REF**: MountingHole_2.2mm_M2_DIN965_Pad_TopBottom, MountingHole:MountingHole_2.2mm_M2_DIN965_Pad_TopBottom, F.Cu at (248.6, 164.4)
- added REF**: M2-COUNTERSUNK, m65_plates_library:M2_Countersunk, F.Cu at (202.8, 150.8)
- added REF**: MountingHole_2.2mm_M2_DIN965_Pad_TopBottom, MountingHole:MountingHole_2.2mm_M2_DIN965_Pad_TopBottom, F.Cu at (75.1, 164.4)
- added REF**: MountingHole_2.2mm_M2_DIN965_Pad, MountingHole:MountingHole_2.2mm_M2_DIN965_Pad, F.Cu at (89.8, 63.2)
- added REF**: M2-COUNTERSUNK, m65_plates_library:M2_Countersunk, F.Cu at (328.3, 110.1)
- added REF**: MountingHole_2.2mm_M2_DIN965_Pad, MountingHole:MountingHole_2.2mm_M2_DIN965_Pad, F.Cu at (51.6, 63.2)
- added REF**: M2-COUNTERSUNK, m65_plates_library:M2_Countersunk, F.Cu at (369.3, 63.2)
- added REF**: MountingHole_2.2mm_M2_DIN965_Pad, MountingHole:MountingHole_2.2mm_M2_DIN965_Pad, F.Cu at (359.0, 63.2)
- added REF**: MountingHole_2.2mm_M2_DIN965_Pad_TopBottom, MountingHole:MountingHole_2.2mm_M2_DIN965_Pad_TopBottom, F.Cu at (161.8, 32.7)
- added REF**: M2-COUNTERSUNK, m65_plates_library:M2_Countersunk, F.Cu at (40.7, 63.2)
- moved GR1 5.30 mm to (136.7, 151.2)
- moved GR2 5.30 mm to (191.7, 151.7)
Other:
- outline, holes or cut-outs redrawn
